File: hardware/EE/design/kicad/ESP32-Solar-Battery/ESP32-Solar-Battery.kicad_pcb (KiCad board)
At the start: 2 copper layers, 100 x 100 mm, 39 parts, among them J202 SolarPanel, J301 LiFePo4_32700, J302 LiFePo4_Ext, Q201 SSM3J332R, Q202 SSM3J332R, Q203 SSM3J332R, Q301 SSM3K333R, Q302 SSM3K333R, U203 MAX809T, U301 HY2112, U401 ESP32-WROOM-32D

Commit message: first layout attempt
Parts:
- removed C301: 0.1uF, Capacitor_SMD:C_0603_1608Metric
- removed D202: BAT54A, Package_TO_SOT_SMD:SOT-23
- removed J301: LiFePo4_32700, ESP32-Solar-Battery:32700_holder
- removed J302: LiFePo4_Ext, Connector_JST:JST_VH_B2P-VH_1x02_P3.96mm_Vertical
- removed Q301, Q302: SSM3K333R, ESP32-Solar-Battery:SOT95P240X88-3N
- removed R301: 2K, Resistor_SMD:R_0603_1608Metric
- removed R302: 100, Resistor_SMD:R_0603_1608Metric
- removed U301: HY2112, Package_TO_SOT_SMD:SOT-23-6
- added C401: 10uF, Capacitor_SMD:C_0603_1608Metric, F.Cu at (105.8, 54.5)
- added C402: 10uF, Capacitor_SMD:C_0603_1608Metric, F.Cu at (113.2, 63.7)
- added C403: 0.1uF, Capacitor_SMD:C_0603_1608Metric, F.Cu at (111.6, 63.7)
- added D1: BZT52C3V9, Diode_SMD:D_SOD-123, F.Cu at (177.7, 86.5)
- added D203: SD103AW, Diode_SMD:D_SOD-123, F.Cu at (104.4, 167.9)
- added D204: SS56, ESP32-Solar-Battery:SOD-128, F.Cu at (90.7, 152.5)
- added D401: LED, LED_SMD:LED_0603_1608Metric, F.Cu at (138.2, 82.1)
- added F201: Fuse, Connector_PinHeader_2.54mm:PinHeader_1x02_P2.54mm_Vertical, F.Cu at (45.1, 68.6)
- added J201: NTC 10K B=3950K, Connector_PinHeader_2.54mm:PinHeader_1x02_P2.54mm_Vertical, F.Cu at (125.5, 137.5)
- added J203: LiFePo4_Batt, Connector_JST:JST_VH_B2P-VH_1x02_P3.96mm_Vertical, F.Cu at (135.6, 132.7)
- added J206: LOAD, Connector_JST:JST_VH_B2P-VH_1x02_P3.96mm_Vertical, F.Cu at (34.9, 60.4)
- added J401: Program, Connector_JST:JST_PH_B3B-PH-K_1x03_P2.00mm_Vertical, F.Cu at (144.9, 57.1)
- added J402: Conn_01x16, Connector_PinHeader_2.54mm:PinHeader_1x16_P2.54mm_Vertical, F.Cu at (102.7, 63.9)
- added J403: Conn_01x16, Connector_PinHeader_2.54mm:PinHeader_1x16_P2.54mm_Vertical, F.Cu at (147.0, 63.1)
- added JP401: RESET, Connector_PinHeader_2.54mm:PinHeader_1x02_P2.54mm_Vertical, F.Cu at (104.1, 57.6)
- added JP402: RESET, Connector_PinHeader_2.54mm:PinHeader_1x02_P2.54mm_Vertical, F.Cu at (137.4, 85.2)
- added L201: 47uH, Inductor_SMD:L_Taiyo-Yuden_NR-80xx_HandSoldering, F.Cu at (98.2, 150.2)
- added Q1: MUN2211T1, Package_TO_SOT_SMD:SC-59, F.Cu at (184.0, 81.2)
- added R213: 39K 1%, Resistor_SMD:R_0603_1608Metric, F.Cu at (119.8, 133.1)
- added R214: 680K, Resistor_SMD:R_0603_1608Metric, F.Cu at (53.0, 39.5)
- added R401: 10K, Resistor_SMD:R_0603_1608Metric, F.Cu at (105.9, 60.6)
- added R402: 220, Resistor_SMD:R_0603_1608Metric, F.Cu at (138.2, 80.3)
- added U201: LMV331, Package_TO_SOT_SMD:SOT-23-5, F.Cu at (125.5, 131.8)
- added U202: CN3801, Package_SO:SSOP-10_3.9x4.9mm_P1.00mm, F.Cu at (98.6, 168.2)
- R202, R204: value 100K -> 100K 1%
- R203: value 8.2K -> 8.2K 1%
- R205: value TBD -> 30K 1%
- R210: value TBD_Rsense -> 0.1; footprint Resistor_SMD:R_0603_1608Metric -> Resistor_SMD:R_2512_6332Metric
- U203: value MAX809T -> IMP810S
- moved C211 138.4 mm to (37.2, 43.5)
- moved R207 128.8 mm to (101.9, 180.3)
- moved R209 124.8 mm to (103.5, 170.8)
- moved C206 123.8 mm to (103.5, 172.5), turned to 180 degrees
- moved C205 121.6 mm to (85.5, 162.0)
- moved R205 121.2 mm to (103.7, 164.0)
- moved R204 118.2 mm to (103.6, 165.7), turned to 180 degrees
- moved D201 113.7 mm to (101.7, 177.1)
- moved Q201 113.1 mm to (92.5, 162.3), turned to 90 degrees
- moved R210 101.0 mm to (109.5, 157.1)
- moved U203 98.9 mm to (53.4, 48.0)
- moved C208 97.6 mm to (117.3, 158.1)
- moved Q203 97.0 mm to (66.6, 36.2)
- moved C209 92.6 mm to (116.4, 154.8)
- moved C207 92.6 mm to (116.1, 161.3)
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Connections:
- C205 pad 2: (no net) -> Net-(C205-Pad2)
- C211 pad 1: (no net) -> VDD_3V2
- Q201 pad 1: (no net) -> Net-(Q201-Pad1)
- Q201 pad 3: (no net) -> Net-(D204-Pad1)
- Q203 pad 3: (no net) -> Net-(F201-Pad2)
- R202 pad 2: Net-(J201-Pad2) -> Net-(R202-Pad2)
- R203 pad 1: Net-(J201-Pad2) -> Net-(R202-Pad2)
- R206 pad 2: (no net) -> Net-(J201-Pad2)
- R209 pad 1: (no net) -> Net-(R209-Pad1)
- R210 pad 1: (no net) -> Net-(L201-Pad2)
- U401 pad 1: Net-(U401-Pad1) -> PB-
- U401 pad 10: (no net) -> ESP32_10
- U401 pad 11: (no net) -> ESP32_11
- U401 pad 12: (no net) -> ESP32_12
- U401 pad 13: (no net) -> ESP32_13
- U401 pad 14: (no net) -> ESP32_14
- U401 pad 15: Net-(U401-Pad1) -> PB-
- U401 pad 16: (no net) -> ESP32_16
- U401 pad 17: (no net) -> Net-(U401-Pad17)
- U401 pad 18: (no net) -> Net-(U401-Pad18)
- U401 pad 19: (no net) -> Net-(U401-Pad19)
- U401 pad 2: (no net) -> VDD_3V2
- U401 pad 20: (no net) -> Net-(U401-Pad20)
- U401 pad 21: (no net) -> Net-(U401-Pad21)
- U401 pad 22: (no net) -> Net-(U401-Pad22)
- U401 pad 23: (no net) -> ESP32_23
- U401 pad 24: (no net) -> ESP32_24
- U401 pad 25: (no net) -> ESP32_25
- U401 pad 26: (no net) -> ESP32_26
- U401 pad 27: (no net) -> ESP32_27
- U401 pad 28: (no net) -> ESP32_28
- U401 pad 29: (no net) -> ESP32_29
- U401 pad 3: (no net) -> ESP32_3
- U401 pad 30: (no net) -> ESP32_30
- U401 pad 31: (no net) -> ESP32_31
- U401 pad 32: (no net) -> Net-(U401-Pad32)
- U401 pad 33: (no net) -> ESP32_33
- U401 pad 34: (no net) -> ESP32_34
- U401 pad 35: (no net) -> ESP32_35
- U401 pad 36: (no net) -> ESP32_36
- U401 pad 37: (no net) -> ESP32_37
- U401 pad 38: Net-(U401-Pad1) -> PB-
- U401 pad 4: (no net) -> ESP32_4
- U401 pad 5: (no net) -> ESP32_5
- U401 pad 6: (no net) -> ESP32_6
- U401 pad 7: (no net) -> ESP32_7
- U401 pad 8: (no net) -> ESP32_8
- U401 pad 9: (no net) -> ESP32_9
Routing:
- net PB+: track 76.9 -> 0.00 mm
- net Net-(C301-Pad2): track 36.0 -> 0.00 mm
- net Net-(J201-Pad2): track 0.00 -> 8.73 mm
- net Net-(R202-Pad2): track 0.00 -> 3.61 mm
Other:
- board size 100 x 100 mm -> 50 x 90 mm

Commit message: Release PCB V1 for fabrication
Parts:
- removed J401: Program, Connector_JST:JST_PH_B3B-PH-K_1x03_P2.00mm_Vertical
- removed JP401, JP402: RESET, Connector_PinHeader_2.54mm:PinHeader_1x02_P2.54mm_Vertical
- added G***: LOGO, ESP32-Solar-Battery:sicris, B.Cu at (125.0, 69.0)
- added J301: Program, Connector_PinHeader_1.27mm:PinHeader_2x03_P1.27mm_Vertical, F.Cu at (127.0, 87.2)
- added J302: jtag, Connector_PinHeader_1.27mm:PinHeader_2x05_P1.27mm_Vertical, F.Cu at (118.4, 87.2)
- added R301: 100, Resistor_SMD:R_0603_1608Metric, F.Cu at (118.4, 90.4)
- added R302: 100, Resistor_SMD:R_0603_1608Metric, F.Cu at (127.0, 90.4)
- moved R214 105.6 mm to (133.7, 107.5), turned to 270 degrees
- moved U203 103.0 mm to (136.9, 108.3), turned to 180 degrees
- moved J206 100.5 mm to (127.5, 99.5), turned to 180 degrees
- moved C211 99.0 mm to (122.8, 93.2), turned to 180 degrees
- moved Q203 95.7 mm to (130.7, 107.2), turned to 90 degrees
- moved F201 86.9 mm to (123.5, 106.1), turned to 90 degrees
- moved R211 71.4 mm to (131.9, 121.8), turned to 180 degrees
- moved Q1 69.4 mm to (129.9, 124.7)
- moved D1 65.0 mm to (128.7, 129.2), turned to 90 degrees
- moved R212 64.3 mm to (134.5, 124.0), turned to 90 degrees
- moved Q202 64.1 mm to (137.3, 122.2), turned to 90 degrees
- moved R207 54.5 mm to (115.7, 127.6)
- moved D201 53.2 mm to (115.7, 125.8)
- moved R204 52.9 mm to (124.2, 116.9)
- moved R205 52.9 mm to (124.2, 115.2)
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Connections:
- net ESP32_13 renamed TMS
- net ESP32_14 renamed TDI
- net ESP32_16 renamed TCK
- net ESP32_23 renamed TDO
- net ESP32_25 renamed BOOT
- net ESP32_3 renamed EN
- net ESP32_34 renamed RXD0
- net ESP32_35 renamed TXD0
- J403 pad 7: Net-(J403-Pad7) -> PB-
- U202 pad 4: Net-(U202-Pad4) -> (no net)
- U401 pad 17: Net-(U401-Pad17) -> (no net)
- U401 pad 18: Net-(U401-Pad18) -> (no net)
- U401 pad 19: Net-(U401-Pad19) -> (no net)
- U401 pad 20: Net-(U401-Pad20) -> (no net)
- U401 pad 21: Net-(U401-Pad21) -> (no net)
- U401 pad 22: Net-(U401-Pad22) -> (no net)
- U401 pad 32: Net-(U401-Pad32) -> (no net)
Routing:
- net VDD_3V2: track 0.00 -> 87.0 mm, vias 0 -> 2
- net Solar_V+: track 0.00 -> 66.1 mm, vias 0 -> 4
- net TXD0: track 0.00 -> 41.8 mm, vias 0 -> 1
- net TDO: track 0.00 -> 41.2 mm
- net EN: track 0.00 -> 40.5 mm, vias 0 -> 1
- net RXD0: track 0.00 -> 37.4 mm, vias 0 -> 1
- net Net-(L201-Pad2): track 0.00 -> 35.3 mm, vias 0 -> 2
- net PB+: track 0.00 -> 34.5 mm
- net TCK: track 0.00 -> 29.7 mm, vias 0 -> 1
- net BOOT: track 0.00 -> 28.4 mm, vias 0 -> 1
- net Net-(C207-Pad1): track 0.00 -> 28.3 mm, vias 0 -> 2
- net TDI: track 0.00 -> 28.2 mm, vias 0 -> 2
- net ESP32_24: track 0.00 -> 26.7 mm
- net TMS: track 0.00 -> 25.2 mm
- net ESP32_26: track 0.00 -> 21.5 mm
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- added copper zone on B.Cu, net Net-(D204-Pad1)
- added copper zone on F.Cu, net Net-(D204-Pad1)
- added copper zone on B.Cu, net PB-
- added copper zone on F.Cu, net PB-
Other:
- board size 50 x 90 mm -> 42 x 79 mm
- board text added: "ESP32 Solar-Battery DevKit v1"
